File: ComputerDesigns/CR2021_CPU_v2/CR2021_CPU_v2.kicad_pcb (KiCad board)
At the start: 2 copper layers, 178.4 x 115.6 mm, 39 parts, among them J1 Conn_02x06_Odd_Even, SW1 RESET, U2 74HCU04, U3 7400, U4 7400, U5 74LS163, Y1 Crystal 8MHz

Commit message: add sound
Parts:
- added $4002: 74LS273, Package_DIP:DIP-20_W7.62mm, F.Cu at (72.9, 56.8)
- added $4003: 74LS273, Package_DIP:DIP-20_W7.62mm, F.Cu at (73.2, 26.6)
- added J3: Conn_STK500v2, Connector_IDC:IDC-Header_2x03_P2.54mm_Vertical, F.Cu at (45.5, 84.9)
- added U6: ATmega328-P, Package_DIP:DIP-28_W7.62mm, F.Cu at (16.0, 50.6)
- R1: value 1k -> 1k
Connections:
- net /R!W renamed R/!W
- net Net-(BUS1-Pin_1) renamed DATA0
- net Net-(BUS1-Pin_2) renamed DATA1
- net Net-(BUS1-Pin_3) renamed DATA2
- net Net-(BUS1-Pin_4) renamed DATA3
- net Net-(BUS1-Pin_5) renamed DATA4
- net Net-(BUS1-Pin_6) renamed DATA5
- net Net-(BUS1-Pin_7) renamed DATA6
- net Net-(BUS1-Pin_8) renamed DATA7
- net Net-(CONN8-Pin_1) renamed $4002_OUT
- net Net-(CONN8-Pin_2) renamed $4003_OUT
Routing:
- net (no net): track 2482.9 -> 2160.0 mm
- net R/!W: track 156.6 -> 0.00 mm
- net CLK: track 57.1 -> 213.7 mm
- net Net-(CONN3-Pin_1): track 0.00 -> 38.7 mm
- net Net-(CONN4-Pin_1): track 0.00 -> 31.9 mm
- net Net-(CONN3-Pin_8): track 0.00 -> 26.9 mm
- net Net-(CONN4-Pin_8): track 0.00 -> 24.8 mm
- net Net-(CONN4-Pin_2): track 0.00 -> 23.0 mm
- net Net-(CONN3-Pin_5): track 0.00 -> 22.5 mm
- net Net-(CONN3-Pin_2): track 0.00 -> 20.2 mm
- net Net-(CONN3-Pin_7): track 0.00 -> 18.1 mm
- net Net-(CONN4-Pin_7): track 0.00 -> 17.0 mm
- net Net-(CONN4-Pin_4): track 0.00 -> 17.0 mm
- net Net-(CONN3-Pin_6): track 0.00 -> 15.6 mm
- net Net-(CONN4-Pin_5): track 0.00 -> 15.0 mm
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
Commit message: update schematics
Parts:
- added LS1: Speaker, Connector_PinHeader_2.54mm:PinHeader_1x02_P2.54mm_Vertical, F.Cu at (69.7, 108.6)
- added U1: LM324, Package_DIP:DIP-14_W7.62mm, F.Cu at (47.4, 108.4)
- added U7: LM324, Package_DIP:DIP-14_W7.62mm, F.Cu at (58.2, 108.4)
- added U8: W65C22NxP, Package_DIP:DIP-40_W15.24mm, F.Cu at (119.7, 190.0)
- J3: value Conn_STK500v2 -> Atmega328 Programmer Interface
- moved $4002 121.5 mm to (139.3, 158.5), turned to 90 degrees
Connections:
- net Net-(IN1-G1) renamed /$4000_IN
- net Net-(IN2-G1) renamed /$4001_IN
- net Net-(J3-MOSI) renamed /Sound/PWM_Sound_Out_Voice2
- net Net-(OUT1-Cp) renamed /$4000_OUT
- net Net-(OUT2-Cp) renamed /$4001_OUT
- net Net-(U6-PD6) renamed /Sound/PWM_Sound_Out_Voice1
- U6 pad 2: Net-($4002-Q6) -> DATA6
- U6 pad 23: Net-($4002-Q0) -> DATA0
- U6 pad 24: Net-($4002-Q1) -> DATA1
- U6 pad 25: Net-($4002-Q2) -> DATA2
- U6 pad 26: Net-($4002-Q3) -> DATA3
- U6 pad 27: Net-($4002-Q4) -> DATA4
- U6 pad 28: Net-($4002-Q5) -> DATA5
- U6 pad 3: Net-($4002-Q7) -> DATA7
- U6 pad 4: Net-($4003-Q0) -> $4002_OUT
- U6 pad 5: Net-($4003-Q1) -> $4003_OUT
- U6 pad 6: R/!W -> unconnected-(U6-PD4-Pad6)
